Commit message: 👌 fix wheel direction

File: urdf/mini_robot_description.urdf (robot description, URDF)
Before this commit: robot mini_robot_description, 3 links, 2 joints
Links:
- removed link leftwheel_link
- removed link rightwheel_link
- added link left_wheel_link, mass 0.026404; collision mesh filename=package://robot_resto_urdf/meshes/right_wheel_link.STL; visual mesh filename=package://robot_resto_urdf/meshes/right_wheel_link.STL
- added link right_wheel_link, mass 0.026404; collision mesh filename=package://robot_resto_urdf/meshes/right_wheel_link.STL; visual mesh filename=package://robot_resto_urdf/meshes/right_wheel_link.STL
- link base_link: geometry collision mesh filename=package://robot_resto_urdf/meshes/base_link.STL; visual mesh filename=package://robot_resto_urdf/meshes/base_link.STL
Joints:
- removed joint leftwheel_joint
- removed joint rightwheel_joint
- added joint left_joint: type continuous, parent base_link, child left_wheel_link, origin xyz=0 0.06726 0.01625 rpy=1.5708 -0.042963 3.1416, axis 0 0 1, limit effort=5 velocity=1.0
- added joint right_joint: type continuous, parent base_link, child right_wheel_link, origin xyz=0 -0.06726 0.01625 rpy=1.5708 0.085809 0, axis 0 0 1, limit effort=5 velocity=1.0
