Commit message: 🚿Cleaning

File: urdf/mini_robot_description.xacro (robot description, xacro)
@@ -5,4 +5,5 @@
 <xacro:include filename="$(find mini_robot_description)/gazebo/mini_robot_description_physics.gazebo" />
 <xacro:include filename="$(find mini_robot_description)/gazebo/mini_robot_description_plugins.gazebo" />
+<xacro:include filename="$(find mini_robot_description)/urdf/materials.xacro" />
 <!-- ############# LINKS ############# -->
   <link name="base_link">
@@ -10,11 +11,5 @@
       <origin xyz="0 0 0" rpy="0 0 0" />
       <mass value="0.62609" />
-      <inertia
-        ixx="0.0011527"
-        ixy="-6.6808E-08"
-        ixz="3.2285E-07"
-        iyy="0.0023193"
-        iyz="-1.2268E-06"
-        izz="0.0012482" />
+      <inertia ixx="0.0011527" ixy="-6.6808E-08" ixz="3.2285E-07" iyy="0.0023193" iyz="-1.2268E-06" izz="0.0012482" />
     </inertial>
     <visual>
@@ -23,8 +18,5 @@
         <mesh  filename="package://mini_robot_description/meshes/base_link.STL" />
       </geometry>
-      <material
-        name="">
-        <color rgba="0.75294 0.75294 0.75294 1" />
-      </material>
+      <material name="white"/>
     </visual>
     <collision>
@@ -39,11 +31,5 @@
       <origin xyz="0 0 0" rpy="0 0 0" />
       <mass value="0.026404" />
-      <inertia
-        ixx="0.0011527"
-        ixy="-6.6808E-08"
-        ixz="3.2285E-07"
-        iyy="0.0023193"
-        iyz="-1.2268E-06"
-        izz="0.0012482" />
+      <inertia  ixx="0.0011527"  ixy="-6.6808E-08"  ixz="3.2285E-07"  iyy="0.0023193"  iyz="-1.2268E-06"  izz="0.0012482" />
     </inertial>
     <visual>
@@ -52,8 +38,5 @@
         <mesh filename="package://mini_robot_description/meshes/right_wheel_link.STL" />
       </geometry>
-      <material
-        name="">
-        <color rgba="0.75294 0.75294 0.75294 1" />
-      </material>
+      <material name="white"/>
     </visual>
     <collision>
@@ -68,11 +51,5 @@
       <origin xyz="0 0 0" rpy="0 0 0" />
       <mass value="0.026404" />
-      <inertia
-        ixx="0.0011527"
-        ixy="-6.6808E-08"
-        ixz="3.2285E-07"
-        iyy="0.0023193"
-        iyz="-1.2268E-06"
-        izz="0.0012482" />
+      <inertia  ixx="0.0011527"  ixy="-6.6808E-08"  ixz="3.2285E-07"  iyy="0.0023193"  iyz="-1.2268E-06"  izz="0.0012482" />
     </inertial>
     <visual>
@@ -81,8 +58,5 @@
         <mesh filename="package://mini_robot_description/meshes/right_wheel_link.STL" />
       </geometry>
-      <material
-        name="">
-        <color rgba="1 1 1 1" />
-      </material>
+      <material name="white"/>
     </visual>
     <collision>
@@ -104,5 +78,5 @@
         <mesh filename="package://mini_robot_description/meshes/lidar.stl" scale="0.001 0.001 0.001"/>
       </geometry>
-      <material name="black"/>
+      <material name="white"/>
     </visual>
     <collision>

Commit message: 🔨 Add Color to RVIZ

File: urdf/mini_robot_description.xacro (robot description, xacro)
@@ -5,5 +5,6 @@
 <xacro:include filename="$(find mini_robot_description)/gazebo/mini_robot_description_physics.gazebo" />
 <xacro:include filename="$(find mini_robot_description)/gazebo/mini_robot_description_plugins.gazebo" />
-<xacro:include filename="$(find mini_robot_description)/urdf/materials.xacro" />
+<!-- ############# Material ############# -->
+<xacro:include filename="$(find mini_robot_description)/urdf/materials.urdf" />
 <!-- ############# LINKS ############# -->
   <link name="base_link">
@@ -38,5 +39,5 @@
         <mesh filename="package://mini_robot_description/meshes/right_wheel_link.STL" />
       </geometry>
-      <material name="white"/>
+      <material name="black"/>
     </visual>
     <collision>
@@ -58,5 +59,5 @@
         <mesh filename="package://mini_robot_description/meshes/right_wheel_link.STL" />
       </geometry>
-      <material name="white"/>
+      <material name="black"/>
     </visual>
     <collision>
@@ -78,5 +79,5 @@
         <mesh filename="package://mini_robot_description/meshes/lidar.stl" scale="0.001 0.001 0.001"/>
       </geometry>
-      <material name="white"/>
+      <material name="blue"/>
     </visual>
     <collision>
