Commit message: 👨🏻‍🏭 Improve move_base problem only in final rotation

File: mini_robot_description/urdf/mini_robot_description.xacro (robot description, xacro)
@@ -11,5 +11,5 @@
     <inertial>
       <origin xyz="0 0 0" rpy="0 0 0" />
-      <mass value="0.62609" />
+      <mass value="5.62609" />
       <inertia ixx="0.0011527" ixy="-6.6808E-08" ixz="3.2285E-07" iyy="0.0023193" iyz="-1.2268E-06" izz="0.0012482" />
     </inertial>
@@ -31,5 +31,5 @@
     <inertial>
       <origin xyz="0 0 0" rpy="0 0 0" />
-      <mass value="0.026404" />
+      <mass value="1.26404" />
       <inertia  ixx="0.0011527"  ixy="-6.6808E-08"  ixz="3.2285E-07"  iyy="0.0023193"  iyz="-1.2268E-06"  izz="0.0012482" />
     </inertial>
@@ -51,5 +51,5 @@
     <inertial>
       <origin xyz="0 0 0" rpy="0 0 0" />
-      <mass value="0.026404" />
+      <mass value="1.26404" />
       <inertia  ixx="0.0011527"  ixy="-6.6808E-08"  ixz="3.2285E-07"  iyy="0.0023193"  iyz="-1.2268E-06"  izz="0.0012482" />
     </inertial>
@@ -71,5 +71,5 @@
     <inertial>
       <origin rpy="0 0 0" xyz="-2.3483549826952554e-09 -3.4770506128023716e-07 0.009561590682608923"/>
-      <mass value="0.0886181648250366"/>
+      <mass value="0.886181648250366"/>
       <inertia ixx="3.3e-05" ixy="0.0" ixz="0.0" iyy="3.3e-05" iyz="0.0" izz="6e-05"/>
     </inertial>

Commit message: 🐛 fix link warning of dummy link in xacro

File: mini_robot_description/urdf/mini_robot_description.xacro (robot description, xacro)
@@ -8,4 +8,5 @@
 <xacro:include filename="$(find mini_robot_description)/urdf/materials.urdf" />
 <!-- ############# LINKS ############# -->
+<link name="dummy"></link>
   <link name="base_link">
     <inertial>
@@ -89,4 +90,8 @@
   </link>
 <!-- ############# JOINTS ############# -->
+  <joint name="dummy_joint" type="fixed">
+     <parent link="dummy"/>
+     <child link="base_link"/>
+   </joint>
   <joint name="right_joint" type="continuous">
     <origin xyz="0 -0.06726 0.01625" rpy="1.5708 0.085809 0" />

Commit message: 🐛 FIX error of redundant TF publish

File: mini_robot_description/urdf/mini_robot_description.xacro (robot description, xacro)
@@ -8,5 +8,5 @@
 <xacro:include filename="$(find mini_robot_description)/urdf/materials.urdf" />
 <!-- ############# LINKS ############# -->
-<link name="dummy"></link>
+<!-- <link name="dummy"></link> -->
   <link name="base_link">
     <inertial>
@@ -90,8 +90,8 @@
   </link>
 <!-- ############# JOINTS ############# -->
-  <joint name="dummy_joint" type="fixed">
+  <!-- <joint name="dummy_joint" type="fixed">
      <parent link="dummy"/>
      <child link="base_link"/>
-   </joint>
+   </joint> -->
   <joint name="right_joint" type="continuous">
     <origin xyz="0 -0.06726 0.01625" rpy="1.5708 0.085809 0" />

Commit message: 🐛 Fix lidar postion and publish + amcl estmiation

File: mini_robot_description/urdf/mini_robot_description.xacro (robot description, xacro)
@@ -69,4 +69,24 @@
     </collision>
   </link>
+  <link name="support_lidar">
+    <inertial>
+      <origin xyz="0 0 0" rpy="0 0 0" />
+      <mass value="0.26" />
+      <inertia ixx="3.3e-05" ixy="0.0" ixz="0.0" iyy="3.3e-05" iyz="0.0" izz="6e-05"/>
+    </inertial>
+    <visual>
+      <origin rpy="0 0 0" xyz="0 0 0"/>
+      <geometry>
+        <cylinder radius="0.04"   length="0.02"/>
+      </geometry>
+      <material name="blue"/>
+    </visual>
+    <collision>
+      <origin rpy="0 0 0" xyz="0 0 0"/>
+      <geometry>
+        <cylinder radius="0.04"   length="0.02"/>
+      </geometry>
+    </collision>
+  </link>
   <link name="lidar_link">
     <inertial>
@@ -110,6 +130,11 @@
     <axis  xyz="0 0 1" />
   </joint>
+  <joint name="support_lidar_joint" type="fixed">
+    <origin xyz="0 0.0 0.14" rpy="0.0 0.0 0.0" />
+    <parent link="base_link" />
+    <child link="support_lidar" />
+  </joint>
   <joint name="lidar_joint" type="fixed">
-    <origin xyz="0 0.0 0.14" rpy="0.0 0.0 0.0" />
+    <origin xyz="0 0.0 0.15" rpy="0.0 0.0 0.0" />
     <parent link="base_link" />
     <child link="lidar_link" />
